Commit message: Rebase from 'upstream'

File: leo_description/urdf/macros.xacro (robot description, xacro)
@@ -7,5 +7,6 @@
                        link_prefix:=''
                        joint_prefix:=''
-                       imu_translation:='0.0628 -0.0314 -0.0393'">
+                       imu_translation:='0.0628 -0.0314 -0.0393'
+                       mecanum_wheels:=false">
     <xacro:macro name="rocker_link" params="name">
       <link name="${link_prefix}rocker_${name}_link">
@@ -60,4 +61,32 @@
           <geometry>
             <mesh filename="package://leo_description/models/Wheel_outline.stl"/>
+          </geometry>
+        </collision>
+      </link>
+    </xacro:macro>
+    <xacro:macro name="mecanum_wheel_link" params="name model">
+      <link name="${link_prefix}wheel_${name}_link">
+        <inertial>
+          <mass value="0.672214"/>
+          <origin xyz="0 -0.036852 0"/>
+          <inertia
+            ixx="0.0009778"  ixy="-8.10228e-7" ixz="3.2e-11"
+            iyy="0.001321" iyz="5.7e-11"
+            izz="0.0009773"/>
+        </inertial>
+        <visual>
+          <geometry>
+            <mesh filename="package://leo_description/models/WheelMecanum${model}.dae"/>
+          </geometry>
+        </visual>
+        <collision>
+          <origin xyz="0 -0.0317 0" rpy="${pi/2} 0 0"/>
+          <geometry>
+            <cylinder radius="0.0635" length="0.0515"/>
+          </geometry>
+        </collision>
+        <collision>
+          <geometry>
+            <mesh filename="package://leo_description/models/Mecanum_wheel_outline.stl"/>
           </geometry>
         </collision>
@@ -90,8 +119,16 @@
     <xacro:rocker_link name="L"/>
     <xacro:rocker_link name="R"/>
-    <xacro:wheel_link name="FL" model="A"/>
-    <xacro:wheel_link name="RL" model="A"/>
-    <xacro:wheel_link name="FR" model="B"/>
-    <xacro:wheel_link name="RR" model="B"/>
+    <xacro:if value="${mecanum_wheels}">
+      <xacro:mecanum_wheel_link name="FL" model="B"/>
+      <xacro:mecanum_wheel_link name="RL" model="A"/>
+      <xacro:mecanum_wheel_link name="FR" model="A"/>
+      <xacro:mecanum_wheel_link name="RR" model="B"/>
+    </xacro:if>
+    <xacro:unless value="${mecanum_wheels}">
+      <xacro:wheel_link name="FL" model="A"/>
+      <xacro:wheel_link name="RL" model="A"/>
+      <xacro:wheel_link name="FR" model="B"/>
+      <xacro:wheel_link name="RR" model="B"/>
+    </xacro:unless>
     <xacro:if value="${default_antenna}">
       <link name="${link_prefix}antenna_link">
@@ -152,5 +189,10 @@
     </joint>
     <joint name="${joint_prefix}wheel_FL_joint" type="continuous">
-      <origin xyz="-0.15256 -0.08214 -0.08802" rpy="0 0 0"/>
+      <xacro:if value="${mecanum_wheels}">
+        <origin xyz="-0.15256 -0.00884 -0.08802" rpy="0 0 0"/>
+      </xacro:if>
+      <xacro:unless value="${mecanum_wheels}">
+        <origin xyz="-0.15256 -0.08214 -0.08802" rpy="0 0 0"/>
+      </xacro:unless>
       <parent link="${link_prefix}rocker_L_link"/>
       <child link="${link_prefix}wheel_FL_link"/>
@@ -160,5 +202,10 @@
     </joint>
     <joint name="${joint_prefix}wheel_RL_joint" type="continuous">
-      <origin xyz="0.15256 -0.08214 -0.08802" rpy="0 0 0"/>
+      <xacro:if value="${mecanum_wheels}">
+        <origin xyz="0.15256 -0.00884 -0.08802" rpy="0 0 0"/>
+      </xacro:if>
+      <xacro:unless value="${mecanum_wheels}">
+        <origin xyz="0.15256 -0.08214 -0.08802" rpy="0 0 0"/>
+      </xacro:unless>
       <parent link="${link_prefix}rocker_L_link"/>
       <child link="${link_prefix}wheel_RL_link"/>
@@ -168,5 +215,10 @@
     </joint>
     <joint name="${joint_prefix}wheel_FR_joint" type="continuous">
-      <origin xyz="0.15256 -0.08214 -0.08802" rpy="0 0 0"/>
+      <xacro:if value="${mecanum_wheels}">
+        <origin xyz="0.15256 -0.00884 -0.08802" rpy="0 0 0"/>
+      </xacro:if>
+      <xacro:unless value="${mecanum_wheels}">
+        <origin xyz="0.15256 -0.08214 -0.08802" rpy="0 0 0"/>
+      </xacro:unless>
       <parent link="${link_prefix}rocker_R_link"/>
       <child link="${link_prefix}wheel_FR_link"/>
@@ -176,5 +228,10 @@
     </joint>
     <joint name="${joint_prefix}wheel_RR_joint" type="continuous">
-      <origin xyz="-0.15256 -0.08214 -0.08802" rpy="0 0 0"/>
+      <xacro:if value="${mecanum_wheels}">
+        <origin xyz="-0.15256 -0.00884 -0.08802" rpy="0 0 0"/>
+      </xacro:if>
+      <xacro:unless value="${mecanum_wheels}">
+        <origin xyz="-0.15256 -0.08214 -0.08802" rpy="0 0 0"/>
+      </xacro:unless>
       <parent link="${link_prefix}rocker_R_link"/>
       <child link="${link_prefix}wheel_RR_link"/>
@@ -208,5 +265,5 @@
   <!-- LEO GAZEBO -->
   <xacro:macro name="leo_gazebo"
-               params="robot_ns:=''">
+               params="robot_ns:='''">
     <xacro:property name="link_prefix" value=""/>
     <xacro:if value="${robot_ns != '' and robot_ns != '/'}">
@@ -215,105 +272,183 @@
     <!-- base ODE properties -->
     <gazebo reference="${link_prefix}base_footprint">
-      <kp>1e6</kp>
-      <kd>1.0</kd>
-      <mu1>0.3</mu1>
-      <mu2>0.3</mu2>
-      <minDepth>0.003</minDepth>
+      <collision>
+        <surface>
+          <friction>
+            <ode>
+              <mu>0.3</mu>
+              <mu2>0.3</mu2>
+            </ode>
+            <bullet>
+              <friction>0.3</friction>
+              <friction2>0.3</friction2>
+              <rolling_friction>0.1</rolling_friction>
+            </bullet>
+          </friction>
+        </surface>
+      </collision>
     </gazebo>
     <gazebo reference="${link_prefix}base_link">
-      <kp>1e6</kp>
-      <kd>1.0</kd>
-      <mu1>0.3</mu1>
-      <mu2>0.3</mu2>
-      <minDepth>0.003</minDepth>
+      <collision>
+        <surface>
+          <friction>
+            <ode>
+              <mu>0.3</mu>
+              <mu2>0.3</mu2>
+            </ode>
+            <bullet>
+              <friction>0.3</friction>
+              <friction2>0.3</friction2>
+              <rolling_friction>0.1</rolling_friction>
+            </bullet>
+          </friction>
+        </surface>
+      </collision>
     </gazebo>
     <!-- rocker ODE properties -->
     <gazebo reference="${link_prefix}rocker_L_link">
-      <kp>1e6</kp>
-      <kd>1.0</kd>
-      <mu1>0.3</mu1>
-      <mu2>0.3</mu2>
-      <minDepth>0.003</minDepth>
+      <collision>
+        <surface>
+          <friction>
+            <ode>
+              <mu>0.3</mu>
+              <mu2>0.3</mu2>
+            </ode>
+            <bullet>
+              <friction>0.3</friction>
+              <friction2>0.3</friction2>
+              <rolling_friction>0.1</rolling_friction>
+            </bullet>
+          </friction>
+        </surface>
+      </collision>
     </gazebo>
     <gazebo reference="${link_prefix}rocker_R_link">
-      <kp>1e6</kp>
-      <kd>1.0</kd>
-      <mu1>0.3</mu1>
-      <mu2>0.3</mu2>
-      <minDepth>0.003</minDepth>
+      <collision>
+        <surface>
+          <friction>
+            <ode>
+              <mu>0.3</mu>
+              <mu2>0.3</mu2>
+            </ode>
+            <bullet>
+              <friction>0.3</friction>
+              <friction2>0.3</friction2>
+              <rolling_friction>0.1</rolling_friction>
+            </bullet>
+          </friction>
+        </surface>
+      </collision>
     </gazebo>
     <!-- wheel ODE properties -->
     <gazebo reference="${link_prefix}wheel_FL_link">
-      <kp>1e6</kp>
-      <kd>100.0</kd>
-      <mu1>3.0</mu1>
-      <mu2>1.0</mu2>
-      <fdir1>1 0 0</fdir1>
-      <minDepth>0.003</minDepth>
+      <collision>
+        <surface>
+          <friction>
+            <ode>
+              <mu>1.0</mu>
+              <mu2>1.0</mu2>
+              <fdir1>0 0 0</fdir1>
+            </ode>
+            <bullet>
+              <friction>1</friction>
+              <friction2>1</friction2>
+              <rolling_friction>0.1</rolling_friction>
+            </bullet>
+          </friction>
+        </surface>
+      </collision>
     </gazebo>
     <gazebo reference="${link_prefix}wheel_FR_link">
-      <kp>1e6</kp>
-      <kd>100.0</kd>
-      <mu1>3.0</mu1>
-      <mu2>1.0</mu2>
-      <fdir1>1 0 0</fdir1>
-      <minDepth>0.003</minDepth>
+      <collision>
+        <surface>
+          <friction>
+            <ode>
+              <mu>1.0</mu>
+              <mu2>1.0</mu2>
+              <fdir1>0 0 0</fdir1>
+            </ode>
+            <bullet>
+              <friction>1</friction>
+              <friction2>1</friction2>
+              <rolling_friction>0.1</rolling_friction>
+            </bullet>
+          </friction>
+        </surface>
+      </collision>
     </gazebo>
     <gazebo reference="${link_prefix}wheel_RL_link">
-      <kp>1e6</kp>
-      <kd>100.0</kd>
-      <mu1>3.0</mu1>
-      <mu2>1.0</mu2>
-      <fdir1>1 0 0</fdir1>
-      <minDepth>0.003</minDepth>
+      <collision>
+        <surface>
+          <friction>
+            <ode>
+              <mu>1.0</mu>
+              <mu2>1.0</mu2>
+              <fdir1>0 0 0</fdir1>
+            </ode>
+            <bullet>
+              <friction>1</friction>
+              <friction2>1</friction2>
+              <rolling_friction>0.1</rolling_friction>
+            </bullet>
+          </friction>
+        </surface>
+      </collision>
     </gazebo>
     <gazebo reference="${link_prefix}wheel_RR_link">
-      <kp>1e6</kp>
-      <kd>100.0</kd>
-      <mu1>3.0</mu1>
-      <mu2>1.0</mu2>
-      <fdir1>1 0 0</fdir1>
-      <minDepth>0.003</minDepth>
+      <collision>
+        <surface>
+          <friction>
+            <ode>
+              <mu>1.0</mu>
+              <mu2>1.0</mu2>
+              <fdir1>0 0 0</fdir1>
+            </ode>
+            <bullet>
+              <friction>1</friction>
+              <friction2>1</friction2>
+              <rolling_friction>0.1</rolling_friction>
+            </bullet>
+          </friction>
+        </surface>
+      </collision>
     </gazebo>
     <!-- camera -->
     <gazebo reference="${link_prefix}camera_frame">
-      <sensor type="camera" name="camera">
-        <always_on>true</always_on>
-        <update_rate>30.0</update_rate>
-        <visualize>false</visualize>
-        <camera name="leo_camera">
-          <horizontal_fov>1.9</horizontal_fov>
-          <image>
-            <width>640</width>
-            <height>480</height>
-            <format>R8G8B8</format>
-          </image>
-          <clip>
-            <near>0.02</near>
-            <far>300</far>
-          </clip>
-          <noise>
-            <type>gaussian</type>
-            <mean>0.0</mean>
-            <stddev>0.007</stddev>
-          </noise>
-          <distortion>
-            <k1>-0.279817</k1>
-            <k2>0.060321</k2>
-            <k3>0.000487</k3>
-            <p1>0.000310</p1>
-            <p2>0.000000</p2>
-            <center>0.5 0.5</center>
-          </distortion>
-        </camera>
-        <plugin name="camera_controller" filename="libgazebo_ros_camera.so">
-          <ros><namespace>${robot_ns}</namespace></ros>
-          <frame_name>camera_optical_frame</frame_name>
-        </plugin>
+      <sensor name="camera" type="camera">
+          <camera name="leo_camera">
+              <horizontal_fov>1.9</horizontal_fov>
+              <image>
+                  <width>640</width>
+                  <height>480</height>
+                  <format>R8G8B8</format>
+              </image>
+              <clip>
+                  <near>0.2</near>
+                  <far>300</far>
+              </clip>
+              <noise>
+                <type>gaussian</type>
+                <mean>0.0</mean>
+                <stddev>0.007</stddev>
+              </noise>
+              <distortion>
+                <k1>-0.279817</k1>
+                <k2>0.060321</k2>
+                <k3>0.000487</k3>
+                <p1>0.000310</p1>
+                <p2>0.000000</p2>
+                <center>0.5 0.5</center>
+              </distortion>
+          </camera>
+          <always_on>1</always_on>
+          <update_rate>30</update_rate>
+          <visualize>true</visualize>
+          <topic>${link_prefix}camera/image_raw</topic>
+          <ignition_frame_id>${link_prefix}camera_frame</ignition_frame_id>
       </sensor>
     </gazebo>
     <!-- rocker differential -->
     <gazebo>
-      <plugin name="rocker_differential" filename="libleo_gazebo_differential_plugin.so">
+      <plugin name="leo_gz::DifferentialSystem" filename="libleo_gz_differential_plugin.so">
         <jointA>rocker_L_joint</jointA>
         <jointB>rocker_R_joint</jointB>
@@ -321,69 +456,43 @@
       </plugin>
     </gazebo>
+    <gazebo>
+      <plugin
+        filename="ignition-gazebo-joint-state-publisher-system"
+        name="ignition::gazebo::systems::JointStatePublisher">
+        <topic>${link_prefix}joint_states</topic>
+      </plugin>
+      <plugin filename="libignition-gazebo-imu-system.so"
+        name="ignition::gazebo::systems::Imu">
+      </plugin>
+    </gazebo>
     <gazebo reference="${link_prefix}imu_frame">
       <sensor type="imu" name="leo_imu_sensor">
         <update_rate>100</update_rate>
-        <plugin filename="libgazebo_ros_imu_sensor.so" name="imu_plugin">
-          <robotNamespace>${robot_ns}</robotNamespace>
-          <topicName>imu/data_raw</topicName>
-          <frameName>${link_prefix}imu_frame</frameName>
-          <updateRateHZ>100.0</updateRateHZ>
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